File: sch/main_board.sch (EAGLE design)
At the start: 0 parts

Commit message: - Add power supply for main board,
Parts:
- added C1, C2, C3, C4, C5: 4.7u, resistor:C-EUC1206
- added D2: VS-10BQ015-M3_5BT, SamacSys_Parts:VS-10BQ015-M3_5BT
- added IC1: MCP73831T-2ACI_OT, SamacSys_Parts:MCP73831T-2ACI_OT
- added J1: MICRO_USB_B_HIROSE_ZX62-B-5PA(11), connector:MICRO_USB_B_HIROSE_ZX62-B-5PA(11)
- added L1: SRN2512-2R2M, SamacSys_Parts:SRN2512-2R2M
- added LED1: GREEN, led:LEDCHIPLED_1206
- added R1: 100k, resistor:R-EU_R1206
- added R2: 10k, resistor:R-EU_R1206
- added R3: 100, resistor:R-EU_R1206
- added R4: 316k, resistor:R-EU_R1206
- added U$1: BAT_FLAT_PAD, connector:BAT_FLAT_PAD
- added U$2: TLV62568DRLT, SamacSys_Parts:TLV62568DRLT
- added U$3: SMAJ5.0A, SamacSys_Parts:SMAJ5.0A
Connections:
- new net GND: C1.2, C2.2, C3.2, C4.2, C5.2, IC1.VSS, J1.GND, R1.1, R2.1, U$1.-, U$2.GND, U$3.A
- new net ID: J1.ID
- new net N$1: LED1.A, R3.1
- new net N$2: IC1.STAT, LED1.C
- new net N$3: IC1.PROG, R2.2
- new net N$6: L1.1, U$2.SW
- new net N$8: R1.2, R4.1, U$2.FB
- new net USB_D+: J1.D+
- new net USB_D-: J1.D-
- new net VCC: C1.1, C5.1, L1.2, R4.2
- new net V_BATT: C2.1, D2.A, IC1.VBAT, U$1.+
- new net V_USB: C3.1, C4.1, D2.K, IC1.VDD, J1.+5V, R3.2, U$2.EN, U$2.VIN, U$3.C
Other:
- note added: "Battery supply"
- note added: "Step-Down 5V - 2.5V"
- note added: "USB connector"
